File: eagle/TF0060DCA.brd (EAGLE design)
At the start: 53.3 x 20.7 mm, 32 parts, among them IC1 LM1972MX_NOPB, IC12 MCP6002T-I_SN, IC2 7805DT, IC3 CH32V203C, IC8 LM1117MPX-3.3

Commit message: Correct C8-C11,C14,C15 value to 10uF as fitted in production (LCSC C1713)
Parts:
- C10, C11, C14, C15, C8, C9: value 6uF -> 10uF
Changed lines of the file:
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@@
 <attribute name="VALUE" x="16.51" y="14.2748" size="1.27" layer="28" rot="MR90" align="center"/>
 </element>
-<element name="C8" library="rcl" library_urn="urn:adsk.eagle:library:334" package="C0805" package3d_urn="urn:adsk.eagle:package:23617/2" value="6uF" x="8.4328" y="6.3276" smashed="yes" rot="MR270">
+<element name="C8" library="rcl" library_urn="urn:adsk.eagle:library:334" package="C0805" package3d_urn="urn:adsk.eagle:package:23617/2" value="10uF" x="8.4328" y="6.3276" smashed="yes" rot="MR270">
 <attribute name="NAME" x="7.7978" y="6.9626" size="0.6096" layer="26" rot="MR270" align="center"/>
 <attribute name="POPULARITY" value="63" x="8.4328" y="6.3276" size="1.778" layer="28" rot="MR270" display="off"/>
@@
 <attribute name="VALUE" x="10.3378" y="6.9626" size="1.27" layer="28" rot="MR270"/>
 </element>
-<element name="C9" library="rcl" library_urn="urn:adsk.eagle:library:334" package="C0805" package3d_urn="urn:adsk.eagle:package:23617/2" value="6uF" x="9.271" y="14.1732" smashed="yes" rot="MR270">
+<element name="C9" library="rcl" library_urn="urn:adsk.eagle:library:334" package="C0805" package3d_urn="urn:adsk.eagle:package:23617/2" value="10uF" x="9.271" y="14.1732" smashed="yes" rot="MR270">
 <attribute name="NAME" x="8.001" y="15.4432" size="0.6096" layer="26" rot="MR270" align="center"/>
 <attribute name="POPULARITY" value="63" x="9.271" y="14.1732" size="1.778" layer="28" rot="MR270" display="off"/>
@@
 <attribute name="VALUE" x="11.811" y="15.4432" size="1.27" layer="28" rot="MR270"/>
 </element>
-<element name="C10" library="rcl" library_urn="urn:adsk.eagle:library:334" package="C0805" package3d_urn="urn:adsk.eagle:package:23617/2" value="6uF" x="14.4526" y="20.0406" smashed="yes" rot="MR0">
+<element name="C10" library="rcl" library_urn="urn:adsk.eagle:library:334" package="C0805" package3d_urn="urn:adsk.eagle:package:23617/2" value="10uF" x="14.4526" y="20.0406" smashed="yes" rot="MR0">
 <attribute name="NAME" x="15.7226" y="21.3106" size="0.6096" layer="26" rot="MR0" align="center"/>
 <attribute name="POPULARITY" value="63" x="14.4526" y="20.0406" size="1.778" layer="28" rot="MR0" display="off"/>
@@
 <attribute name="VALUE" x="15.7226" y="17.5006" size="1.27" layer="28" rot="MR0"/>
 </element>
-<element name="C11" library="rcl" library_urn="urn:adsk.eagle:library:334" package="C0805" package3d_urn="urn:adsk.eagle:package:23617/2" value="6uF" x="12.5222" y="5.4864" smashed="yes" rot="MR180">
+<element name="C11" library="rcl" library_urn="urn:adsk.eagle:library:334" package="C0805" package3d_urn="urn:adsk.eagle:package:23617/2" value="10uF" x="12.5222" y="5.4864" smashed="yes" rot="MR180">
 <attribute name="NAME" x="11.2522" y="4.2164" size="0.6096" layer="26" rot="MR180" align="center"/>
 <attribute name="POPULARITY" value="63" x="12.5222" y="5.4864" size="1.778" layer="28" rot="MR180" display="off"/>
@@
 <attribute name="VALUE" x="11.2522" y="8.0264" size="1.27" layer="28" rot="MR180"/>
 </element>
-<element name="C14" library="rcl" library_urn="urn:adsk.eagle:library:334" package="C0805" package3d_urn="urn:adsk.eagle:package:23617/2" value="6uF" x="14.3002" y="8.8392" smashed="yes" rot="MR180">
+<element name="C14" library="rcl" library_urn="urn:adsk.eagle:library:334" package="C0805" package3d_urn="urn:adsk.eagle:package:23617/2" value="10uF" x="14.3002" y="8.8392" smashed="yes" rot="MR180">
 <attribute name="NAME" x="13.0302" y="7.5692" size="1.27" layer="26" rot="MR180"/>
 <attribute name="POPULARITY" value="63" x="14.3002" y="8.8392" size="0.6096" layer="28" rot="MR180" display="off"/>
@@
 <attribute name="VALUE" x="13.0302" y="11.3792" size="1.27" layer="28" rot="MR180"/>
 </element>
-<element name="C15" library="rcl" library_urn="urn:adsk.eagle:library:334" package="C0805" package3d_urn="urn:adsk.eagle:package:23617/2" value="6uF" x="12.192" y="14.1732" smashed="yes" rot="MR270">
+<element name="C15" library="rcl" library_urn="urn:adsk.eagle:library:334" package="C0805" package3d_urn="urn:adsk.eagle:package:23617/2" value="10uF" x="12.192" y="14.1732" smashed="yes" rot="MR270">
 <attribute name="NAME" x="10.922" y="15.4432" size="1.27" layer="26" rot="MR270"/>
 <attribute name="POPULARITY" value="63" x="12.192" y="14.1732" size="0.6096" layer="28" rot="MR270" display="off"/>
